Commit message: my_arm

File: my_robotic_arm1/src/mrm_desp/src/urdf/mrm.urdf (robot description, URDF)
Before this commit: robot mrm, 6 links, 5 joints
Links:
- removed link link_3
- removed link link_4
- removed link link_5
Joints:
- removed joint joint_3
- removed joint joint_4
- removed joint joint_5
